File: V1-root/V1-main/V1.kicad_pcb (KiCad board)
At the start: 2 copper layers, 208 parts, among them J1 OLED, J2 Conn_01x03_Socket, J3 DebugSTM, M1 Motor_DC, M2 Motor_DC, Q1 PMOS, Q10 NMOS, Q11 NMOS, Q2 AO3400A, Q3 AO3400A, Q4 NMOS, Q5 NMOS, Q6 NMOS, Q7 NMOS, Q8 NMOS, Q9 NMOS, SW1 SW_SPST, U1 AP64500SP-3.3v, U10 UCC27211ADRMR_C, U11 UCC27211ADRMR_A, U12 LM393, U13 LM393, U14 LM393, U15 LM393, U16 LM393, U17 LM393, U18 UCC27211ADRMR_D, U19 UCC27211ADRMR_B, U2 STM32G431C6T6, U20 XIAO-ESP32-S3-DIP_ui, U21 4053, U22 4053, U3 STM32G491RET6, U4 LM393, U5 LM393, U6 LM393, U7 LM393, U8 LM393, U9 LM393, Y1 Crystal_GND24, Y2 Crystal_GND24

Commit message: footprint紐付け&pcb同期
Parts:
- removed D14: D_Schottky, Diode_THT:D_A-405_P10.16mm_Horizontal
- added LED_15: LED, LED_SMD:LED_0603_1608Metric_Pad1.05x0.95mm_HandSolder, F.Cu at (87.2, 50.0)
- added LED_16: LED, LED_SMD:LED_0603_1608Metric_Pad1.05x0.95mm_HandSolder, F.Cu at (87.2, 52.6)
- added R66: 10k, Resistor_SMD:R_0603_1608Metric_Pad0.98x0.95mm_HandSolder, F.Cu at (36.3, 52.2)
- added R67: 10k, Resistor_SMD:R_0603_1608Metric_Pad0.98x0.95mm_HandSolder, F.Cu at (36.3, 54.7)
- added R68: 10m, FC4L110R005FER:FC4L110_OHM, F.Cu at (64.8, 80.1)
- added R69: 10m, FC4L110R005FER:FC4L110_OHM, F.Cu at (73.1, 80.1)
- added U23: 4053, 74HC4053PW:SOT403-1_NXP, F.Cu at (95.6, 104.6)
- added slide2: SW_SPDT, Connector_PinSocket_2.54mm:PinSocket_1x03_P2.54mm_Vertical, F.Cu at (57.4, 23.9)
- added tact_4: SW_Push, 74th:Switch_SKRPABE010, F.Cu at (20.4, 107.2)
- added togg2: SW_SPDT, Connector_PinSocket_2.54mm:PinSocket_1x03_P2.54mm_Vertical, F.Cu at (66.6, 23.9)
- J3: value DebugSTM -> Conn_01x04_Socket; footprint Connector_PinSocket_2.54mm:PinSocket_1x07_P2.54mm_Vertical -> Connector_PinSocket_2.54mm:PinSocket_1x04_P2.54mm_Vertical
- R10, R47: footprint Resistor_THT:R_Axial_DIN0207_L6.3mm_D2.5mm_P10.16mm_Horizontal -> Resistor_SMD:R_0603_1608Metric
- R11: value 220 -> 10k; footprint Resistor_SMD:R_0805_2012Metric -> Resistor_THT:R_Axial_DIN0207_L6.3mm_D2.5mm_P10.16mm_Horizontal
- R12, R40: value 25 -> 220; footprint Resistor_SMD:R_0603_1608Metric -> Resistor_SMD:R_0805_2012Metric
- R14, R17: value 12.5 -> 25
- R15: value 25 -> 12.5
- R18: value 10k -> 12.5
- R19: value 3.3k -> 10k; footprint Resistor_THT:R_Axial_DIN0207_L6.3mm_D2.5mm_P10.16mm_Horizontal -> Resistor_SMD:R_0603_1608Metric
- R20: value 10k -> 3.3k; footprint Resistor_SMD:R_0603_1608Metric -> Resistor_THT:R_Axial_DIN0207_L6.3mm_D2.5mm_P10.16mm_Horizontal
- R21, R43: value 1k -> 10k
- R23, R30: value 69.8k -> 1k
- R28, R35: value 1k -> 69.8k
- R39: value 220 -> 1k; footprint Resistor_SMD:R_0805_2012Metric -> Resistor_SMD:R_0603_1608Metric
- R42: value 10k -> 25
- R48, R49: value 4.7 -> 1k; footprint Resistor_SMD:R_0603_1608Metric_Pad0.98x0.95mm_HandSolder -> Resistor_THT:R_Axial_DIN0207_L6.3mm_D2.5mm_P10.16mm_Horizontal
- R50, R51: value 4.7 -> 470; footprint Resistor_SMD:R_0603_1608Metric_Pad0.98x0.95mm_HandSolder -> Resistor_SMD:R_0603_1608Metric
- R52, R53, R54, R55, R60, R61, R62, R63: value 10k -> 4.7
- R56, R57, R58, R59: value 4.7 -> 10k
- R64, R65: value 10m -> 10k; footprint FC4L110R005FER:FC4L110_OHM -> Resistor_SMD:R_0603_1608Metric_Pad0.98x0.95mm_HandSolder
- R9: value 10k -> 1k; footprint Resistor_SMD:R_0603_1608Metric -> Resistor_THT:R_Axial_DIN0207_L6.3mm_D2.5mm_P10.16mm_Horizontal
- U20: value XIAO-ESP32-S3-DIP_ui -> AT25SF321B-SSHB-B; footprint Seeed Xiao:XIAO-ESP32-S3-DIP -> AT25SF321B-SSHB:SOIC127P599X175-8N
- tact_1, tact_2: footprint Button_Switch_THT:SW_PUSH-12mm -> Button_Switch_THT:SW_TH_Tactile_Omron_B3F-10xx
- tact_3: footprint Button_Switch_THT:SW_PUSH-12mm -> 74th:Switch_SKRPABE010
- moved D1 87.7 mm to (72.4, 103.6)
- moved R3 87.7 mm to (71.1, 106.3)
- moved slide1 78.1 mm to (52.8, 23.9)
- moved togg1 77.9 mm to (62.0, 23.9)
- moved tact_2 75.8 mm to (93.1, 30.9)
- moved tact_1 75.6 mm to (93.1, 23.2)
- moved Q1 71.9 mm to (56.6, 35.3)
- moved U2 71.7 mm to (44.1, 102.0)
- moved Multiplex_1 71.0 mm to (87.1, 64.8)
- moved BZ1 69.3 mm to (84.2, 94.5)
- moved C35 68.3 mm to (57.6, 91.3)
- moved C36 68.3 mm to (57.6, 93.3)
- moved C37 68.3 mm to (57.6, 95.3)
- moved C8 68.3 mm to (57.6, 89.4)
- moved C38 68.3 mm to (57.6, 97.3)
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Connections:
- net SPI_CS renamed SPI_CS_MCU
- C55 pad 1: GND -> VCC
- C55 pad 2: +3.3V -> GND
- C57 pad 1: VCC -> +3.3V
- J3 pad 2: SWD_IO -> X
- J3 pad 3: SWD_CLK -> Y
- R10 pad 1: VCC -> PWM_line
- R10 pad 2: VOUT -> PWM
- R11 pad 1: Net-(Q2-G) -> VCC
- R11 pad 2: BRIGHTNESS -> VOUT
- R12 pad 1: +3.3V -> Net-(Q2-G)
- R12 pad 2: Net-(LED_1-A) -> BRIGHTNESS
- R13 pad 2: Net-(LED_3-A) -> Net-(LED_1-A)
- R14 pad 2: Net-(LED_5-A) -> Net-(LED_3-A)
- R15 pad 2: Net-(LED_6-A) -> Net-(LED_5-A)
- R16 pad 2: Net-(LED_8-A) -> Net-(LED_6-A)
- R17 pad 2: Net-(LED_10-A) -> Net-(LED_8-A)
- R18 pad 1: GND -> +3.3V
- R18 pad 2: Net-(Q2-G) -> Net-(LED_10-A)
- R19 pad 1: VOUT -> GND
- R19 pad 2: GND -> Net-(Q2-G)
- R20 pad 1: PWM_encorder -> VOUT
- R20 pad 2: ENCORDER_PWM -> GND
- R21 pad 1: encorderDigi_R -> PWM_encorder
- R21 pad 2: +3.3V -> ENCORDER_PWM
- R22 pad 1: Net-(R22-Pad1) -> encorderDigi_R
- R23 pad 1: /mark_A -> Net-(R23-Pad1)
- R23 pad 2: GND -> +3.3V
- R24 pad 1: /mark_B -> /mark_A
- R25 pad 1: /mark_C -> /mark_B
- R26 pad 1: /mark_D -> /mark_C
- R27 pad 1: encorderADC_R -> /mark_D
- R28 pad 1: encorderDigi_L -> encorderADC_R
- R28 pad 2: +3.3V -> GND
- R29 pad 1: Net-(R29-Pad1) -> encorderDigi_L
- R30 pad 1: encorderADC_L -> Net-(R30-Pad1)
- R30 pad 2: GND -> +3.3V
- R31 pad 1: /goal_A -> encorderADC_L
- R32 pad 1: /goal_B -> /goal_A
- R33 pad 1: /goal_C -> /goal_B
- R34 pad 1: /goal_D -> /goal_C
- R35 pad 1: A_mark -> /goal_D
- R35 pad 2: +3.3V -> GND
- R36 pad 1: B_mark -> A_mark
- R37 pad 1: C_mark -> B_mark
- R38 pad 1: D_mark -> C_mark
- R39 pad 1: Net-(Q3-G) -> D_mark
- R39 pad 2: EBRIGHTNESS -> +3.3V
- R40 pad 1: +3.3V -> Net-(Q3-G)
- R40 pad 2: Net-(LED_11-A) -> EBRIGHTNESS
- R41 pad 2: Net-(LED_13-A) -> Net-(LED_11-A)
- R42 pad 1: GND -> +3.3V
- R42 pad 2: Net-(Q3-G) -> Net-(LED_13-A)
- R43 pad 1: A_goal -> GND
- R43 pad 2: +3.3V -> Net-(Q3-G)
- R44 pad 1: B_goal -> A_goal
- R45 pad 1: C_goal -> B_goal
- R46 pad 1: D_goal -> C_goal
- R47 pad 1: +3.3V -> D_goal
- R47 pad 2: sig -> +3.3V
- R48 pad 1: HO_A -> +3.3V
- R48 pad 2: HS_A -> sig
- R49 pad 1: HS_B -> +3.3V
- R49 pad 2: HO_B -> sig_B
- R50 pad 1: HO_C -> +3.3V
- R50 pad 2: HS_C -> Net-(LED_15-A)
- R51 pad 1: HS_D -> +3.3V
- R51 pad 2: HO_D -> Net-(LED_16-A)
- R52 pad 1: HS_A -> HO_A
- R52 pad 2: Net-(M1-+) -> HS_A
- R53 pad 1: Net-(M1--) -> HS_B
- R53 pad 2: HS_B -> HO_B
- R54 pad 1: HS_C -> HO_C
- R54 pad 2: Net-(M2-+) -> HS_C
- R55 pad 1: Net-(M2--) -> HS_D
- R55 pad 2: HS_D -> HO_D
- R56 pad 1: LO_A -> HS_A
- R56 pad 2: Net-(Q8-G) -> Net-(M1-+)
- R57 pad 1: Net-(Q9-G) -> Net-(M1--)
- R57 pad 2: LO_B -> HS_B
- R58 pad 1: LO_C -> HS_C
- R58 pad 2: Net-(Q10-G) -> Net-(M2-+)
- R59 pad 1: Net-(Q11-G) -> Net-(M2--)
- R59 pad 2: LO_D -> HS_D
- R60 pad 1: Net-(Q8-G) -> LO_A
- R60 pad 2: Net-(Q8-S) -> Net-(Q8-G)
- R61 pad 1: Net-(Q8-S) -> Net-(Q9-G)
- R61 pad 2: Net-(Q9-G) -> LO_B
- R62 pad 1: Net-(Q10-G) -> LO_C
- R62 pad 2: Net-(Q10-S) -> Net-(Q10-G)
- R63 pad 1: Net-(Q10-S) -> Net-(Q11-G)
- R63 pad 2: Net-(Q11-G) -> LO_D
- R64 pad 1: Net-(Q8-S) -> Net-(Q8-G)
- R64 pad 2: shunt_AB -> Net-(Q8-S)
- R65 pad 1: Net-(Q10-S) -> Net-(Q8-S)
- R65 pad 2: shunt_CD -> Net-(Q9-G)
- R8 pad 2: start -> slide
- R9 pad 1: PWM_line -> +3.3V
- R9 pad 2: PWM -> start
- U20 pad 1: tact_3 -> SPI_CS_FLASH
- U20 pad 2: tact_2 -> SPI_MISO
- U20 pad 3: tact_1 -> +3.3V
- U20 pad 4: start -> GND
- U20 pad 5: SDA_OLED -> SPI_MOSI
- U20 pad 6: SCL_OLED -> SPI_SCK
- U20 pad 7: mRXcTX -> +3.3V
- U20 pad 8: mTXcRX -> +3.3V
- U22 pad 1: /sRXlinkTX -> /sTXlinkRX
- U22 pad 12: /mNRST -> /mRXlinkTX
- U22 pad 13: /sNRST -> /sRXlinkTX
- U22 pad 14: NRST -> RXlinkTX
- U22 pad 15: RXlinkTX -> TXlinkRX
- U22 pad 2: /mRXlinkTX -> /mTXlinkRX
- U22 pad 3: /sTXlinkRX -> unconnected-(U22-Z1-Pad3)
- U22 pad 4: TXlinkRX -> unconnected-(U22-Z-Pad4)
- U22 pad 5: /mTXlinkRX -> unconnected-(U22-Z0-Pad5)
- U3 pad 2: unconnected-(U3-PC13-Pad2) -> slide
- U3 pad 24: unconnected-(U3-PB0-Pad24) -> Buzzer
- U3 pad 3: unconnected-(U3-PC14-Pad3) -> tact_1
- U3 pad 34: unconnected-(U3-PB12-Pad34) -> SPI_CS_FLASH
- U3 pad 4: unconnected-(U3-PC15-Pad4) -> tact_2
- U3 pad 54: unconnected-(U3-PC12-Pad54) -> start
- U5 pad 1: Net-(R22-Pad1) -> Net-(R23-Pad1)
- U7 pad 1: Net-(R29-Pad1) -> Net-(R30-Pad1)
- slide1 pad 3: unconnected-(slide1-C-Pad3) -> Net-(LED_15-K)
- tact_3 pad 1: tact_3 -> /mNRST
- togg1 pad 1: start -> slide

Commit message: sideLine配線&MD系配置終了
Parts:
- removed the U4 at (20.9, 24.8)
- removed the U5 at (20.9, 31.2)
- removed the U6 at (20.9, 37.7)
- removed the U7 at (29.4, 24.8)
- removed the U8 at (29.4, 31.2)
- removed the U9 at (29.4, 37.7)
- added F1: Fuse, Fuse:Fuseholder_Clip-5x20mm_Keystone_3517_Inline_P23.11x6.76mm_D1.70mm_Horizontal, F.Cu at (190.5, 144.7)
- added slidemain1: SW_SPDT, 74th:SLIDE_akiduki, F.Cu at (216.5, 150.4)
- C10: footprint Capacitor_SMD:CP_Elec_4x5.4 -> Capacitor_SMD:C_0603_1608Metric_Pad1.08x0.95mm_HandSolder
- C11: footprint Capacitor_SMD:CP_Elec_5x5.7 -> Capacitor_SMD:C_1206_3216Metric
- C5, C6, C7: footprint Capacitor_SMD:CP_Elec_5x5.4 -> Capacitor_SMD:C_0805_2012Metric
- D10, D11, D12, D13, D4, D5, D6, D7, LED_1, LED_10, LED_2, LED_3, LED_4, LED_5, LED_6, LED_7, LED_8, LED_9: moved to B.Cu
- slide1, slide2, togg1, togg2: footprint Connector_PinSocket_2.54mm:PinSocket_1x03_P2.54mm_Vertical -> 74th:SLIDE_akiduki
- moved FB2 243.2 mm to (-29.5, 277.4), turned to 180 degrees
- moved U14 236.9 mm to (272.7, 68.5), turned to -165 degrees
- moved C25 229.8 mm to (-29.6, 275.9)
- moved M1 228.4 mm to (311.3, 114.4)
- moved C32 226.4 mm to (-24.9, 283.4), turned to 180 degrees
- moved R18 225.4 mm to (279.0, 68.8), turned to 105 degrees
- moved U15 219.9 mm to (261.1, 71.6), turned to -165 degrees
- moved R32 216.9 mm to (278.3, 65.9), turned to 15 degrees
- moved Q5 214.8 mm to (229.5, 129.8)
- moved R17 213.2 mm to (266.7, 69.0), turned to 105 degrees
- moved C13 212.7 mm to (227.1, 98.3)
- moved C48 212.6 mm to (229.0, 120.4)
- moved C17 210.6 mm to (228.2, 87.4)
- moved Q9 210.4 mm to (229.5, 136.8)
- moved R44 210.3 mm to (275.8, 71.2), turned to -165 degrees
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- renumbered U22 to U10, U23 to U11, U10 to U4, U11 to U5, U18 to U6, U19 to U7, U20 to U8, U21 to U9
Connections:
- U12 pad 1: C_mark -> A_mark
- U12 pad 3: /mark_C -> /mark_A
- U12 pad 4: (no net) -> GND
- U12 pad 5: (no net) -> /mark_B
- U12 pad 6: (no net) -> PWM
- U12 pad 7: (no net) -> B_mark
- U12 pad 8: (no net) -> +3.3V
- U13 pad 1: D_mark -> C_mark
- U13 pad 3: /mark_D -> /mark_C
- U13 pad 4: (no net) -> GND
- U13 pad 5: (no net) -> /mark_D
- U13 pad 6: (no net) -> PWM
- U13 pad 7: (no net) -> D_mark
- U13 pad 8: (no net) -> +3.3V
- U14 pad 4: (no net) -> GND
- U14 pad 5: (no net) -> /goal_B
- U14 pad 6: (no net) -> PWM
- U14 pad 7: (no net) -> B_goal
- U14 pad 8: (no net) -> +3.3V
- U15 pad 1: B_goal -> C_goal
- U15 pad 3: /goal_B -> /goal_C
- U15 pad 4: (no net) -> GND
- U15 pad 5: (no net) -> /goal_D
- U15 pad 6: (no net) -> PWM
- U15 pad 7: (no net) -> D_goal
- U15 pad 8: (no net) -> +3.3V
- U16 pad 1: C_goal -> encorderDigi_R
- U16 pad 2: PWM -> ENCORDER_PWM
- U16 pad 3: /goal_C -> encorderADC_R
- U16 pad 4: (no net) -> GND
- U16 pad 5: (no net) -> GND
- U16 pad 6: (no net) -> ENCORDER_PWM
- U16 pad 7: (no net) -> Net-(R23-Pad1)
- U16 pad 8: (no net) -> +3.3V
- U17 pad 1: D_goal -> encorderDigi_L
- U17 pad 2: PWM -> ENCORDER_PWM
- U17 pad 3: /goal_D -> encorderADC_L
- U17 pad 4: (no net) -> GND
- U17 pad 5: (no net) -> GND
- U17 pad 6: (no net) -> ENCORDER_PWM
- U17 pad 7: (no net) -> Net-(R30-Pad1)
- U17 pad 8: (no net) -> +3.3V
Routing:
- net LED_GND: track 0.00 -> 73.9 mm, vias 0 -> 3
- net +3.3V: track 0.00 -> 65.1 mm, vias 0 -> 18
- net PWM: track 0.00 -> 62.3 mm, vias 0 -> 2
- net GND: track 0.00 -> 38.8 mm, vias 0 -> 7
- net A_mark: track 0.00 -> 34.0 mm, vias 0 -> 1
- net B_mark: track 0.00 -> 32.7 mm, vias 0 -> 1
- net A_goal: track 0.00 -> 29.4 mm, vias 0 -> 1
- net B_goal: track 0.00 -> 26.9 mm, vias 0 -> 1
- net C_mark: track 0.00 -> 21.8 mm, vias 0 -> 1
- net D_mark: track 0.00 -> 17.9 mm, vias 0 -> 2
- net C_goal: track 0.00 -> 16.2 mm, vias 0 -> 1
- net D_goal: track 0.00 -> 15.4 mm
- net Net-(LED_8-A): track 0.00 -> 12.1 mm, vias 0 -> 2
- net /goal_B: track 0.00 -> 9.32 mm, vias 0 -> 2
- net Net-(LED_3-A): track 0.00 -> 8.30 mm, vias 0 -> 1
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- added copper zone on F.Cu, net +3.3V
- added copper zone on B.Cu, net GND
Other:
- board outline added: 160.8 x 97.7 mm
